File: Hardware Files/A1-Main-Board/A1-Main-Board.kicad_pcb (KiCad board)
At the start: 2 copper layers, 43 parts, among them J1 MotorJST, J11 FPC2, J115 BOOT, J2 MotorJST, J3 MotorJST, J9 FPC1, Q1 NMOS, U1 TMC2209-LA, U105 STM32G431RBT3, U2 TMC2209-LA, U3 TMC2209-LA, U4 AMS1117-3.3, Y103 Crystal_GND24

Commit message: e
e
Parts:
- removed C145, C146: 30pF, Capacitor_SMD:C_0402_1005Metric
- removed C147, C148, C149, C154, C155, C156, C157: 100nF, Capacitor_SMD:C_0402_1005Metric
- removed C150: 10uF, Capacitor_SMD:C_0603_1608Metric
- removed C151: 10nF, Capacitor_SMD:C_0402_1005Metric
- removed C152, C153: 1uF, Capacitor_SMD:C_0201_0603Metric
- removed C17, C7, C9: 100uF, Capacitor_SMD:CP_Elec_8x10
- removed D5, D6: BAV99, Package_TO_SOT_SMD:SOT-23
- removed FB102: 120r 100MHz, Capacitor_SMD:C_0603_1608Metric
- removed J115: BOOT, Connector_PinHeader_2.54mm:PinHeader_1x03_P2.54mm_Vertical
- removed J2, J3: MotorJST, Connector_JST:JST_XH_B4B-XH-A_1x04_P2.50mm_Vertical
- removed Q1: NMOS, Package_TO_SOT_SMD:SOT-23-3
- removed R138: 10kR, Resistor_SMD:R_0402_1005Metric
- removed R28: 10R, Resistor_SMD:R_0402_1005Metric
- removed R30: 20kR, Resistor_SMD:R_0402_1005Metric
- removed R50, R53: 4.7kR, Resistor_SMD:R_0402_1005Metric
- removed R51, R52, R54, R55: 2.37kR, Resistor_SMD:R_0402_1005Metric
- removed U1, U2, U3: TMC2209-LA, footprints:TMC2209-LA
- removed U105: STM32G431RBT3, Package_QFP:LQFP-64_10x10mm_P0.5mm
- removed U4: AMS1117-3.3, Package_TO_SOT_SMD:SOT-223-3_TabPin2
- removed Y103: Crystal_GND24, Crystal:Crystal_SMD_3225-4Pin_3.2x2.5mm
- added A1: RaspberryPi_Pico, Module:RaspberryPi_Pico_Common_THT, F.Cu at (37.3, 156.3)
- added C35: 100uF, Capacitor_SMD:CP_Elec_8x10, F.Cu at (144.5, 159.7)
- added C36: 100uF, Capacitor_SMD:CP_Elec_8x10, F.Cu at (144.5, 170.4)
- added C39: 100uF, Capacitor_SMD:CP_Elec_8x10, F.Cu at (49.0, 164.9)
- added C42: 1uF, PCM_JLCPCB:C_0402, F.Cu at (50.8, 149.8)
- added C43: 1uF, PCM_JLCPCB:C_0402, F.Cu at (56.2, 148.7)
- added C47: 10nF, Capacitor_SMD:C_0402_1005Metric, F.Cu at (58.0, 150.6)
- added C48: 1uF, Capacitor_SMD:C_0201_0603Metric, F.Cu at (57.0, 150.6)
- added C51: 10uF, Capacitor_SMD:C_0603_1608Metric, F.Cu at (97.5, 164.6)
- added C52: 100uF, Capacitor_SMD:CP_Elec_8x10, F.Cu at (94.7, 187.2)
- added C53: 100nF, Capacitor_SMD:C_0402_1005Metric, F.Cu at (67.0, 164.6)
- added C54: 10uF, Capacitor_SMD:C_0603_1608Metric, F.Cu at (65.7, 164.5)
- added C55: 100uF, Capacitor_SMD:CP_Elec_8x10, F.Cu at (66.5, 187.1)
- added C56: 100nF, Capacitor_SMD:C_0402_1005Metric, F.Cu at (83.5, 164.9)
- added C57: 10uF, Capacitor_SMD:C_0603_1608Metric, F.Cu at (82.0, 164.7)
- added C58: 100uF, Capacitor_SMD:CP_Elec_8x10, F.Cu at (82.2, 187.1)
- added C59: 100nF, PCM_JLCPCB:C_0402, F.Cu at (55.3, 144.5)
- added C60: 100nF, PCM_JLCPCB:C_0402, F.Cu at (61.4, 144.5)
- added D1: BAV99, Package_TO_SOT_SMD:SOT-23, F.Cu at (53.5, 142.5)
- added D2: BAV99, Package_TO_SOT_SMD:SOT-23, F.Cu at (59.8, 142.5)
- added FB2: 120r 100MHz, Capacitor_SMD:C_0603_1608Metric, F.Cu at (59.3, 150.2)
- added J10: FPC_CON, Connector_FFC-FPC:Hirose_FH12-8S-0.5SH_1x08-1MP_P0.50mm_Horizontal, F.Cu at (126.5, 186.2)
- added J13: Power-Input, TerminalBlock:TerminalBlock_MaiXu_MX126-5.0-02P_1x02_P5.00mm, F.Cu at (40.2, 167.1)
- added J14: Power-Input, TerminalBlock:TerminalBlock_MaiXu_MX126-5.0-02P_1x02_P5.00mm, F.Cu at (117.3, 187.1)
- added J17: Motor Connector, Connector_JST:JST_XH_B4B-XH-A_1x04_P2.50mm_Vertical, F.Cu at (153.3, 186.0)
- added J18: Motor Connector, Connector_JST:JST_XH_B4B-XH-A_1x04_P2.50mm_Vertical, F.Cu at (57.4, 175.5)
- added J19: Motor Connector, Connector_JST:JST_XH_B4B-XH-A_1x04_P2.50mm_Vertical, F.Cu at (140.1, 186.4)
- added J8: USB_Toolhead_Outgoing, Connector_USB:USB_B_Lumberg_2411_02_Horizontal, F.Cu at (138.0, 168.1)
- added P1: USB_Toolhead_Incoming, Connector_USB:USB_C_Receptacle_HRO_TYPE-C-31-M-12, F.Cu at (154.3, 165.2)
- added R32: 2.2kΩ, PCM_JLCPCB:R_0402, F.Cu at (53.8, 145.0)
- added R33: 2.2kΩ, PCM_JLCPCB:R_0402, F.Cu at (51.7, 145.0)
- added R34: 2.2kΩ, PCM_JLCPCB:R_0402, F.Cu at (58.1, 145.0)
- added R35: 2.2kΩ, PCM_JLCPCB:R_0402, F.Cu at (60.0, 145.0)
- added R38: 10kΩ, PCM_JLCPCB:R_0402, F.Cu at (107.3, 183.0)
- added R39: 10kΩ, PCM_JLCPCB:R_0402, F.Cu at (75.3, 183.2)
- added R40: 10kΩ, PCM_JLCPCB:R_0402, F.Cu at (89.5, 183.2)
- added R41: 4.7kΩ, PCM_JLCPCB:R_0402, F.Cu at (51.2, 143.6)
- added R42: 4.7kΩ, PCM_JLCPCB:R_0402, F.Cu at (57.6, 143.6)
- added U10: TMC2209_SILENTSTEPSTICK, MODULE_TMC2209_SILENTSTEPSTICK:MODULE_TMC2209_SILENTSTEPSTICK, F.Cu at (69.6, 172.1)
- added U11: TMC2209_SILENTSTEPSTICK, MODULE_TMC2209_SILENTSTEPSTICK:MODULE_TMC2209_SILENTSTEPSTICK, F.Cu at (85.5, 172.1)
- added U7: TLV75733PDBV, Package_TO_SOT_SMD:SOT-23-5, F.Cu at (53.5, 149.3)
- added U9: TMC2209_SILENTSTEPSTICK, MODULE_TMC2209_SILENTSTEPSTICK:MODULE_TMC2209_SILENTSTEPSTICK, F.Cu at (101.5, 172.1)
- C49: value 100nF -> 1uF; footprint Capacitor_SMD:C_0402_1005Metric -> Capacitor_SMD:C_0201_0603Metric
- J1: value MotorJST -> MB_UART
- J11: value FPC2 -> Bed-Binder; footprint Connector_PinHeader_2.54mm:PinHeader_1x08_P2.54mm_Vertical -> Connector_PinHeader_2.54mm:PinHeader_2x08_P2.54mm_Vertical
- J9: value FPC1 -> Toolhead_USB; footprint Connector_PinHeader_2.54mm:PinHeader_1x08_P2.54mm_Vertical -> Connector_JST:JST_XH_B4B-XH-A_1x04_P2.50mm_Vertical
- moved J11 120.3 mm to (113.4, 179.8), turned to 90 degrees
- moved C49 109.9 mm to (58.7, 148.1), turned to 180 degrees
- moved C50 100.8 mm to (98.8, 164.6), turned to 90 degrees
- moved J9 100.2 mm to (153.9, 155.6), turned to 90 degrees
- moved J1 19.2 mm to (39.6, 173.5), turned to -90 degrees
Connections:
- C49 pad 1: /heated-bed/BED_THERM_1 -> +3V3
- C50 pad 1: /heated-bed/BED_THERM_2 -> +3V3
- J1 pad 1: Net-(J1-Pin_1) -> GND
- J1 pad 2: Net-(J1-Pin_2) -> /mcu-pico-tht/UART_RX
- J1 pad 3: Net-(J1-Pin_3) -> /mcu-pico-tht/UART_TX
- J1 pad 4: Net-(J1-Pin_4) -> +3V3
- J11 pad 1: +5V -> Net-(J10-Pin_1)
- J11 pad 2: /heated-bed/100k_THB_INP -> +5V
- J11 pad 3: GND -> Net-(J10-Pin_2)
- J11 pad 4: /heated-bed/10k_THB_INP -> /heated-bed/100k_THB_INP
- J11 pad 5: GND -> Net-(J10-Pin_3)
- J11 pad 6: 5v -> GND
- J11 pad 7: /heated-bed/HEATED_BED- -> Net-(J10-Pin_4)
- J11 pad 8: GND -> /heated-bed/10k_THB_INP
- J9 pad 1: Net-(J8-Pin_1) -> VBUS
- J9 pad 2: Net-(J8-Pin_2) -> /communications-toolhead/USB_D+
- J9 pad 3: Net-(J8-Pin_3) -> /communications-toolhead/USB_D-
- J9 pad 4: Net-(J8-Pin_4) -> GND
Other:
- board outline added: 122.7 x 60 mm
- board text added: "UART OUT"
- board text added: "X MOTOR"
- board text added: "Z MOTOR"
