File: Hardware Files/A1-Main-Board/A1-Main-Board.kicad_pcb (KiCad board)
At the start: 2 copper layers, 122.7 x 60 mm, 47 parts, among them J1 MB_UART, J10 FPC_CON, J11 Bed-Binder, J13 Power-Input, J14 Power-Input, J17 Motor Connector, J18 Motor Connector, J19 Motor Connector, J8 USB_Toolhead_Outgoing, J9 Toolhead_USB, P1 USB_Toolhead_Incoming, U10 TMC2209_SILENTSTEPSTICK, U11 TMC2209_SILENTSTEPSTICK, U7 TLV75733PDBV, U9 TMC2209_SILENTSTEPSTICK

Commit message: e
e
Parts:
- removed C60: 100nF, PCM_JLCPCB:C_0402
- removed D2: BAV99, Package_TO_SOT_SMD:SOT-23
- removed R34, R35: 2.2kΩ, PCM_JLCPCB:R_0402
- removed R42: 4.7kΩ, PCM_JLCPCB:R_0402
- added H1: M1.5, MountingHole:MountingHole_2.2mm_M2_ISO14580_Pad_TopBottom, F.Cu at (2.17, 2.17)
- added H2: M1.5, MountingHole:MountingHole_2.2mm_M2_ISO14580_Pad_TopBottom, F.Cu at (2.17, 7.53)
- added H3: M1.5, MountingHole:MountingHole_2.2mm_M2_ISO14580_Pad_TopBottom, F.Cu at (7.53, 2.17)
- added H4: M1.5, MountingHole:MountingHole_2.2mm_M2_ISO14580_Pad_TopBottom, F.Cu at (7.53, 7.53)
- added H5: M1.5, MountingHole:MountingHole_2.2mm_M2_ISO14580_Pad_TopBottom, F.Cu at (12.9, 2.17)
- added H6: M1.5, MountingHole:MountingHole_2.2mm_M2_ISO14580_Pad_TopBottom, F.Cu at (12.9, 7.53)
- added J12: MotorJST, Connector_JST:JST_XH_B4B-XH-A_1x04_P2.50mm_Vertical, F.Cu at (215.5, 151.5)
- added J15: ExpansionPortJST, Connector_JST:JST_XH_B4B-XH-A_1x04_P2.50mm_Vertical, F.Cu at (2.98, 13.6)
- moved J18 149.3 mm to (144.2, 54.0), turned to 0 degrees
- moved C52 107.8 mm to (161.2, 102.3)
- moved J19 107.4 mm to (198.0, 96.0), turned to -90 degrees
- moved C58 106.5 mm to (146.7, 102.4)
- moved C55 106.0 mm to (130.2, 102.4)
- moved J17 105.9 mm to (210.0, 96.5), turned to -90 degrees
- moved C56 105.7 mm to (146.6, 80.1)
- moved C50 105.7 mm to (161.8, 79.8)
- moved C51 105.7 mm to (160.6, 79.8)
- moved C53 105.7 mm to (130.1, 79.8)
- moved C54 105.7 mm to (128.7, 79.7)
- moved C57 105.7 mm to (145.1, 79.9)
- moved R38 105.7 mm to (170.3, 98.2)
- moved R39 105.7 mm to (138.4, 98.4)
- moved R40 105.7 mm to (152.6, 98.4)
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Connections:
- A1 pad 32: /heated-bed/BED_THERM_2 -> /mcu-pico-tht/BED_THERM2
- J10 pad 1: Net-(J10-Pin_1) -> unconnected-(J10-Pin_1-Pad1)
- J10 pad 2: Net-(J10-Pin_2) -> unconnected-(J10-Pin_2-Pad2)
- J10 pad 3: Net-(J10-Pin_3) -> unconnected-(J10-Pin_3-Pad3)
- J10 pad 4: Net-(J10-Pin_4) -> unconnected-(J10-Pin_4-Pad4)
- J10 pad 5: Net-(J10-Pin_5) -> unconnected-(J10-Pin_5-Pad5)
- J10 pad 6: Net-(J10-Pin_6) -> unconnected-(J10-Pin_6-Pad6)
- J10 pad 7: Net-(J10-Pin_7) -> unconnected-(J10-Pin_7-Pad7)
- J10 pad 8: Net-(J10-Pin_8) -> unconnected-(J10-Pin_8-Pad8)
- J11 pad 1: Net-(J10-Pin_1) -> unconnected-(J11-Pin_1-Pad1)
- J11 pad 11: Net-(J10-Pin_6) -> unconnected-(J11-Pin_11-Pad11)
- J11 pad 12: /heated-bed/HEATED_BED_PWM -> unconnected-(J11-Pin_12-Pad12)
- J11 pad 13: Net-(J10-Pin_7) -> unconnected-(J11-Pin_13-Pad13)
- J11 pad 15: Net-(J10-Pin_8) -> unconnected-(J11-Pin_15-Pad15)
- J11 pad 3: Net-(J10-Pin_2) -> unconnected-(J11-Pin_3-Pad3)
- J11 pad 4: /heated-bed/100k_THB_INP -> unconnected-(J11-Pin_4-Pad4)
- J11 pad 5: Net-(J10-Pin_3) -> unconnected-(J11-Pin_5-Pad5)
- J11 pad 7: Net-(J10-Pin_4) -> unconnected-(J11-Pin_7-Pad7)
- J11 pad 9: Net-(J10-Pin_5) -> unconnected-(J11-Pin_9-Pad9)
Other:
- board size 122.7 x 60 mm -> 176.9 x 142.5 mm
