File: Hardware Files/A1-Main-Board/A1-Main-Board.kicad_sch (KiCad schematic)
At the start: 1 part, among them J1 MB_UART

Commit message: e
e
Parts:
- added H1, H2, H3, H4, H5, H6: M1.5, MountingHole:MountingHole_2.2mm_M2_ISO14580_Pad_TopBottom, symbol Mechanical:MountingHole_Pad
- added J15: ExpansionPortJST, Connector_JST:JST_XH_B4B-XH-A_1x04_P2.50mm_Vertical, symbol Connector_Generic:Conn_01x04
- J1: now not fitted; now left out of the parts list
Other:
- removed sheet power
