File: Hardware Files/A1-Main-Board/comms-toolhead.kicad_sch (KiCad schematic)
At the start: 3 parts, among them J4 UART_PINS, J5 USB_PINS, P1 USB_C_Plug

Commit message: e
e
Parts:
- removed J4: UART_PINS, symbol Connector_Generic:Conn_01x02
- removed J5: USB_PINS, symbol Connector_Generic:Conn_01x02
- added C35, C36: 100uF, Capacitor_SMD:CP_Elec_8x10, symbol Device:C_Polarized
- added J8: USB_Toolhead_Outgoing, Connector_USB:USB_B_Lumberg_2411_02_Horizontal, symbol Connector:USB_B
- added J9: Toolhead_USB, Connector_JST:JST_XH_B4B-XH-A_1x04_P2.50mm_Vertical, symbol Connector_Generic:Conn_01x04
- P1: value USB_C_Plug -> USB_Toolhead_Incoming; footprint (none) -> Connector_USB:USB_C_Receptacle_HRO_TYPE-C-31-M-12
Connections:
- net +24V: now also C35.1
- net +5V: now also C36.1
- net GND: now also C35.2, C36.2, J8.4 (GND), J9.4 (Pin_4)
- net USB_D+: now also J8.3 (D+), J9.2 (Pin_2)
- net USB_D-: now also J8.2 (D-), J9.3 (Pin_3)
- new net VBUS: J8.1 (VBUS), J9.1 (Pin_1)
Other:
- note added: "Toolhead Outgoing"
- note removed: "BACKUP TO CM4"
- note removed: "BACKUP TO RPZ2"
- note removed: "TO CM4"
- note removed: "TO RPZ2"
