File: Hardware Files/A1-Main-Board/drivers.kicad_sch (KiCad schematic)
At the start: 0 parts

Commit message: e
e
Parts:
- added R10: 1k, symbol Device:R
Connections:
- net MA_UART: now also R10.1
- new net UART_RX: R10.2
Other:
- added sheet stepstick-slot (stepstick-slot.kicad_sch)
- added sheet stepstick-slot1 (stepstick-slot.kicad_sch)
- added sheet stepstick-slot2 (stepstick-slot.kicad_sch)
- note added: "Confirm direction"
