File: Hardware Files/A1-Main-Board/fan.kicad_sch (KiCad schematic)
At the start: 0 parts

Commit message: e
e
Changed lines of the file:
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@@
 (kicad_sch
-	(version 20250114)
+	(version 20260306)
 	(generator "eeschema")
-	(generator_version "9.0")
+	(generator_version "10.0")
 	(paper "A4")
 	(hierarchical_label "MB_FAN_PWM"
 		(shape input)
 		(at 137.16 81.28 180)
+		(effects
+			(font
+				(size 1.27 1.27)
+			)
+			(justify right)
+		)
+	)
+	(hierarchical_label "SPARE_FAN_TACH"
+		(shape input)
+		(at 137.16 90.17 180)
 		(effects
 			(font
@@
 		(effects
 			(font
+				(size 1.27 1.27)
+			)
+			(justify right)
+		)
+	)
+	(hierarchical_label "SPARE_FAN_PWM"
+		(shape input)
+		(at 137.16 87.63 180)
+		(effects
+			(font
