File: Hardware Files/A1-Main-Board/mcu.kicad_sch (KiCad schematic)
At the start: 21 parts, among them J115 BOOT, J6 MB_UART, J7 MB_USB, SW101 SW_SPST, U105 STM32G431RBT3, Y103 Crystal_GND24

Commit message: e
e
Parts:
- renumbered C145 to C22, C157 to C23, C146 to C24, C156 to C25, C155 to C26, C148 to C27, C154 to C28, C147 to C29, C149 to C30, C150 to C31, C151 to C32, C152 to C33, C153 to C34, FB102 to FB1, J115 to J5, J7 to J6, J6 to J7, R138 to R29, SW101 to SW1, U105 to U4, Y103 to Y1
