File: Hardware Files/A1-Main-Board/power.kicad_sch (KiCad schematic)
At the start: 3 parts, among them J10 Screw_Terminal_01x02, U4 AMS1117-3.3

Commit message: e
e
Parts:
- removed F1: Fuse, symbol Device:Fuse
- removed J10: Screw_Terminal_01x02, symbol Connector:Screw_Terminal_01x02
- removed U4: AMS1117-3.3, Package_TO_SOT_SMD:SOT-223-3_TabPin2, symbol Regulator_Linear:AMS1117-3.3
- added C39: 100uF, Capacitor_SMD:CP_Elec_8x10, symbol Device:C_Polarized
- added C42, C43: 1uF, PCM_JLCPCB:C_0402, symbol PCM_JLCPCB-Capacitors:0402,1uF
- added J13, J14: Power-Input, TerminalBlock:TerminalBlock_MaiXu_MX126-5.0-02P_1x02_P5.00mm, symbol Connector:Screw_Terminal_01x02
- added U7: TLV75733PDBV, Package_TO_SOT_SMD:SOT-23-5, symbol Regulator_Linear:TLV75733PDBV
Connections:
- net +24V: now also J14.2 (Pin_2)
- net +3V3: now also C43.1, U7.5 (OUT)
- net +5V: now also C39.1, J13.2 (Pin_2)
- net GND: now also C39.2, C42.1, C43.2, J13.1 (Pin_1), J14.1 (Pin_1), U7.2 (GND)
- new net VBUS: C42.2, U7.1 (IN), U7.3 (EN)
