File: Hardware Files/A1-Main-Board/stepstick.kicad_sch (KiCad schematic)
At the start: 18 parts, among them J1 MotorJST, U1 TMC2209-LA

Commit message: e
e
Parts:
- renumbered C7 to C2, C6 to C3, C5 to C4, C4 to C5, C3 to C6, C2 to C7, J1 to J2, R8 to R1, R3 to R2, R4 to R3, R7 to R4, R6 to R5, R5 to R6, R9 to R7, R1 to R8, R2 to R9
