File: Hardware Files/A1-Toolhead-Board/fans.kicad_sch (KiCad schematic)
At the start: 14 parts, among them J4 EXF_PW_JMP, J5 PCF_PW_JMP, J6 EXF, J7 PCF

Commit message: Just chucked whatever is here
Going on holidays and just have an old version but this is backup skibidi 67
Other:
- note added: "some caps seems unneccesary, do i remove for simplicity"
Changed lines of the file:
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@@
+		)
+	)
+	(text "some caps seems unneccesary, do i remove for simplicity"
+		(exclude_from_sim no)
+		(at 147.574 39.878 0)
+		(effects
+			(font
+				(size 1.27 1.27)
+			)
 		)
 	)

Commit message: e
e
Parts:
- removed C13, C27: 4.7uF 50V, Capacitor_SMD:C_1206_3216Metric, symbol Device:C
- removed D1, D2: D, Diode_SMD:D_SOD-123F, symbol Device:D
- removed R21, R23, R24, R242: 10k, Resistor_SMD:R_0402_1005Metric, symbol Device:R
- removed R22, R25: 4.7k, Resistor_SMD:R_0402_1005Metric, symbol Device:R
- added C11, C12: 4.7uF, PCM_JLCPCB:C_1206, symbol PCM_JLCPCB-Capacitors:1206,4.7uF
- added D1, D4: DSK26, PCM_JLCPCB:D_SOD-123FL, symbol PCM_JLCPCB-Diodes:Schottky,DSK26
- added R19, R20, R24, R25: 10kΩ, PCM_JLCPCB:R_0402, symbol PCM_JLCPCB-Resistors:0402,10kΩ
- added R23, R31: 4.7kΩ, PCM_JLCPCB:R_0402, symbol PCM_JLCPCB-Resistors:0402,4.7kΩ
Connections:
- net +24V: now also C12.1, D1.1
- net +3V3: now also R19.2, R24.2
- net EXTR_FAN_PWM: now also R23.1
- net EXTR_FAN_TACH: now also R20.1
- net GND: now also C11.2, C12.2, D1.2, D4.2, R23.2, R31.2
- net PART_FAN_PWM: now also R31.1
- net PART_FAN_TACH: now also R25.1
- net VBUS: now also C11.1, D4.1
- net at J6.2 (Pin_2): now also R19.1, R20.2
- net at J7.1 (Pin_1): now also R24.1, R25.2
- no-connect marks 2 -> 1
Other:
- note added: "1206"
- note added: "do i add custom fan voltage selection? if i have room."
- note added: "do they have too high resistors (does pwm need a current resistor)"
- note removed: "C29823"
- note removed: "C64898"
- company: (none) -> Trihexangular Studios
- title: (none) -> Fans
