File: Hardware Files/A1-Toolhead-Board/heaters.kicad_sch (KiCad schematic)
At the start: 11 parts, among them J11 HT_THO, J8 SGDBM-08-020P-H40, Q1 NMOS

Commit message: Just chucked whatever is here
Going on holidays and just have an old version but this is backup skibidi 67
Other:
- note added: "do i split to 2x 1x02, but too high chance of messing up unless jstph"
- note added: "just copied schematic from skr pico lol"
- note added: "try and get sgdbm for v2, or atleast consign part next order, or get sims_60 to do it."
Changed lines of the file:
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@@
+		)
+	)
+	(text "try and get sgdbm for v2, or atleast consign part next order, or get sims_60 to do it."
+		(exclude_from_sim no)
+		(at 141.986 140.97 0)
+		(effects
+			(font
+				(size 1.27 1.27)
+			)
 		)
 	)
@@
 		)
 	)
+	(text "do i split to 2x 1x02, but too high chance of messing up unless jstph"
+		(exclude_from_sim no)
+		(at 148.59 59.436 0)
+		(effects
+			(font
+				(size 1.27 1.27)
+			)
+		)
+	)
 	(text "Too high resistor? 10k?"
 		(exclude_from_sim no)
@@
 		(effects
 			(font
+				(size 1.27 1.27)
+			)
+		)
+	)
+	(text "just copied schematic from skr pico lol\n"
+		(exclude_from_sim no)
+		(at 108.204 119.634 0)
+		(effects
+			(font

Commit message: e
e
Parts:
- removed C102: 100uF 50V, Capacitor_SMD:CP_Elec_8x10.5, symbol Device:C_Polarized
- removed C12: 100nF, Capacitor_SMD:C_0402_1005Metric, symbol Device:C
- removed J11: HT_THO, Connector_JST:JST_XH_B4B-XH-A_1x04_P2.50mm_Vertical, symbol Connector_Generic:Conn_01x04
- removed Q1: NMOS, Library:PPAK-8L-NumberingFixed, symbol Simulation_SPICE:NMOS
- removed R16: 10R, Resistor_SMD:R_0402_1005Metric, symbol Device:R
- removed R17: 20kR, Resistor_SMD:R_0402_1005Metric, symbol Device:R
- removed R18: 4.7kR, Resistor_SMD:R_0402_1005Metric, symbol Device:R
- removed R19, R20: 2.37kR, Resistor_SMD:R_0402_1005Metric, symbol Device:R
- added C1: 100nF, PCM_JLCPCB:C_0402, symbol PCM_JLCPCB-Capacitors:0402,100nF,(2)
- added J12: THO, Connector_JST:JST_XH_B2B-XH-A_1x02_P2.50mm_Vertical, symbol Connector_Generic:Conn_01x02
- added J13: HE, Connector_JST:JST_XH_B2B-XH-A_1x02_P2.50mm_Vertical, symbol Connector_Generic:Conn_01x02
- added Q2: AO3400A, PCM_JLCPCB:Q_SOT-23, symbol PCM_JLCPCB-Transistors:NMOS,AO3400A
- added R16: 4.7kΩ, PCM_JLCPCB:R_0402, symbol PCM_JLCPCB-Resistors:0402,4.7kΩ
- added R17, R18: 2.2kΩ, Resistor_SMD:R_0603_1608Metric, symbol PCM_JLCPCB-Resistors:0402,2.2kΩ
- added R27: 10Ω, PCM_JLCPCB:R_0402, symbol PCM_JLCPCB-Resistors:0402,10Ω
- added R30: 10kΩ, PCM_JLCPCB:R_0402, symbol PCM_JLCPCB-Resistors:0402,10kΩ
Connections:
- net +24V: now also J13.2 (Pin_2); no longer J8.1 (Pin_1), J8.18 (Pin_18), J8.19 (Pin_19), J8.2 (Pin_2), J8.20 (Pin_20), J8.3 (Pin_3)
- net +3.3VADC: now also R16.1
- net GND: now also C1.2, J12.2 (Pin_2), Q2.2 (S), R30.1; no longer J8.14 (Pin_14), J8.15 (Pin_15), J8.6 (Pin_6), J8.7 (Pin_7)
- net HOTEND_PWM: now also R27.2, R30.2
- net THERMISTER: now also C1.1, R17.1
- net at D3.3 (K): now also R17.2, R18.1
- new net: J13.1 (Pin_1), Q2.3 (D)
- new net: J12.1 (Pin_1), R16.2, R18.2
- new net: Q2.1 (G), R27.1
- now unconnected: J8.10 (Pin_10), J8.11 (Pin_11), J8.12 (Pin_12), J8.13 (Pin_13), J8.16 (Pin_16), J8.17 (Pin_17), J8.4 (Pin_4), J8.5 (Pin_5), J8.8 (Pin_8), J8.9 (Pin_9)
Other:
- note added: "0603 C4190"
- note added: "AO3400A"
- note added: "C20917"
- note added: "should this be >0402?"
- note removed: "C358116"
- note removed: "PPAK-8L"
- note removed: "Too high resistor? 10k?"
- note removed: "do i split to 2x 1x02, but too high chance of messing up unless jstph"
- note removed: "try and get sgdbm for v2, or atleast consign part next order, or get sims_60 to do it."
- company: (none) -> Trihexangular Studios
- title: (none) -> Hotend and Thermister
- moved on the sheet: D3
