File: Hardware Files/A1-Toolhead-Board/mcu.kicad_sch (KiCad schematic)
At the start: 16 parts, among them J2 BOOT, J3 SWDEBUG, SW1 SW_SPST, U2 STM32G431KBU3, Y1 Crystal_GND24

Commit message: Just chucked whatever is here
Going on holidays and just have an old version but this is backup skibidi 67
Parts:
- SW1: footprint A1KLibrary:A Stupid Button -> Connector_PinHeader_2.54mm:PinHeader_1x02_P2.54mm_Vertical
Changed lines of the file:
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@@
 			)
 		)
-		(property "Footprint" "A1KLibrary:A Stupid Button"
+		(property "Footprint" "Connector_PinHeader_2.54mm:PinHeader_1x02_P2.54mm_Vertical"
 			(at 81.28 82.55 0)
 			(effects

Commit message: e
e
Parts:
- removed C16, C17, C22: 100nF, Capacitor_SMD:C_0402_1005Metric, symbol Device:C
- removed C18: 10uF, Capacitor_SMD:C_0603_1608Metric, symbol Device:C
- removed C19: 10nF, Capacitor_SMD:C_0402_1005Metric, symbol Device:C
- removed C20, C21: 1uF, Capacitor_SMD:C_0201_0603Metric, symbol Device:C
- removed C23, C24: 30pF, Capacitor_SMD:C_0402_1005Metric, symbol Device:C
- removed R11: 10kR, Resistor_SMD:R_0402_1005Metric, symbol Device:R
- added C16, C25, C8: 100nF, PCM_JLCPCB:C_0402, symbol PCM_JLCPCB-Capacitors:0402,100nF,(2)
- added C17, C18: 1uF, PCM_JLCPCB:C_0402, symbol PCM_JLCPCB-Capacitors:0402,1uF
- added C19: 10uF, PCM_JLCPCB:C_0603, symbol PCM_JLCPCB-Capacitors:0603,10uF
- added C20: 10nF, PCM_JLCPCB:C_0402, symbol PCM_JLCPCB-Capacitors:0402,10nF
- added C22, C23: 30pF, PCM_JLCPCB:C_0402, symbol PCM_JLCPCB-Capacitors:0402,30pF
- added R11, R7: 10kΩ, PCM_JLCPCB:R_0402, symbol PCM_JLCPCB-Resistors:0402,10kΩ
Connections:
- net FILA_SENSOR_1ADC is gone; now on net BIQU_BL_PROBE: U2.7 (PA2)
- net FILA_SENSOR_2 is gone; now on net BIQU_BL_SERVO: U2.8 (PA3)
- net +3V3: now also C16.1, C17.1, C19.1, C25.1, C8.1, R11.1
- net +3V3A: now also C18.1, C20.1
- net BIQU_BL_PROBE: no longer U2.6 (PA1)
- net BIQU_BL_SERVO: no longer U2.5 (PA0)
- net EXF_FAN_PWM: now also U2.9 (PA4); no longer U2.28 (PB5)
- net EXF_FAN_TACH: now also U2.10 (PA5); no longer U2.29 (PB6)
- net EXTRUDER_DIAG: now also U2.28 (PB5); no longer U2.10 (PA5)
- net EXTRUDER_DIR: now also U2.5 (PA0); no longer U2.12 (PA7)
- net EXTRUDER_ENABLE: now also U2.29 (PB6); no longer U2.11 (PA6)
- net EXTRUDER_STEP: now also U2.27 (PB4); no longer U2.13 (PB0)
- net GND: now also C16.2, C17.2, C18.2, C19.2, C20.2, C22.2, C23.2, C25.2, C8.2
- net PART_FAN_PWM: now also U2.12 (PA7); no longer U2.26 (PB3)
- net PART_FAN_TACH: now also U2.13 (PB0); no longer U2.27 (PB4)
- net THERMISTER: now also U2.11 (PA6); no longer U2.9 (PA4)
- net at U2.2 (PF0), Y1.1: now also C23.1
- net at SW1.2 (B), U2.4 (PG10): now also R11.2
- net at J2.2 (Pin_2): now also R7.1
- net at U2.31 (PB8): now also R7.2
- net at U2.3 (PF1), Y1.3: now also C22.1
- new net FILAMENT_SENSOR: U2.26 (PB3)
Other:
- note added: "STM32F401KBU6"
- note added: "STM32G431KBU3 - Backup, high temp out of stock"
- moved on the sheet: FB1
