File: Hardware Files/A1-Toolhead-Board/rfs.kicad_sch (KiCad schematic)
At the start: 1 part, among them J14 Conn_01x08_Pin

Commit message: e
e
Parts:
- added J11: EXTR_FIL, Connector_PinHeader_2.54mm:PinHeader_1x02_P2.54mm_Vertical, symbol Connector_Generic:Conn_01x02
- added U6: 74LVC1G17, PCM_JLCPCB:SOT-23-5_L3.0-W1.7-P0.95-LS2.8-BR, symbol 74xGxx:74LVC1G17
- J14: value Conn_01x08_Pin -> FPC_FILAMENT_SENSOR; footprint Connector_FFC-FPC:Amphenol_F32Q-1A7x1-11008_1x08-1MP_P0.5mm_Horizontal -> Connector_FFC-FPC:Hirose_FH12-8S-0.5SH_1x08-1MP_P0.50mm_Horizontal
Connections:
- net +3V3: now also J14.1 (Pin_1), J14.2 (Pin_2), U6.5 (VCC); no longer J14.7 (Pin_7), J14.8 (Pin_8)
- net GND: now also J14.7 (Pin_7), J14.8 (Pin_8), U6.3 (GND); no longer J14.3 (Pin_3)
- net SNS1: now also J14.3 (Pin_3), J11.1 (Pin_1); no longer J14.4 (Pin_4)
- net SNS2: now also J11.2 (Pin_2)
- net SNS3: now also U6.2
- new net ADC: U6.4
Other:
- note added: "C7836"
- note removed: "Assumption about filament sensor pinout"
- title: (none) -> Filament Sensor
