File: Hardware Files/A1-Toolhead-Board/A1-Toolhead-Board.kicad_sch (KiCad schematic)
At the start: 1 part

Commit message: Just chucked whatever is here
Going on holidays and just have an old version but this is backup skibidi 67
Parts:
- added H1, H2, H3: m1.5, Library:MountingHole_M1.5, symbol Mechanical:MountingHole_Pad
Connections:
- new net: H1.1, H2.1, H3.1
Other:
- note added: "do i?"

Commit message: e
e
Other:
- removed sheet sensors
- sheet mcu ports: added FILAMENT_SENSOR; removed FILA_SENSOR_1ADC, FILA_SENSOR_2
- sheet reversed_filament_sensor ports: added ADC; removed none
- note added: "100R C25076 0402"
- note added: "100nF 50V C307331 0402"
- note added: "100uF 50V C3352 D8xL10.2mm EXTENDED"
- note added: "200mR C411236 1206 EXTENDED EXPENSIVE"
- note added: "20kR C25545 0402"
- note added: "22nF Something"
- note added: "4.7uF smth"
- note added: "8P FPC - C66953"
- note added: "Components:"
- note added: "TMC2209-LA C2150710"
- moved on the sheet: H1, H2, H3

Commit message: e
e
Connections:
- now unconnected: H1.1, H2.1, H3.1
Changed lines of the file:
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@@
-		(color 0 0 0 0)
-	)
-	(junction
-		(at 99.06 160.02)
-		(diameter 0)
 		(color 0 0 0 0)
 	)
@@
 		)
 		(stroke
-			(width 0)
-			(type default)
-		)
-	)
-	(wire
-		(pts
-			(xy 99.06 160.02) (xy 99.06 166.37)
-		)
-		(stroke
-			(width 0)
-			(type default)
-		)
-	)
-	(wire
-		(pts
-			(xy 99.06 153.67) (xy 99.06 160.02)
-		)
-		(stroke
