File: Hardware Files/A1-Toolhead-Board/A1-Toolhead-Board.kicad_pcb (KiCad board)
At the start: 2 copper layers, 61 parts, among them J1 Motor_E, J10 BL_PROBE, J11 HT_THO, J14 Conn_01x08_Pin, J2 BOOT, J6 EXF, J7 PCF, J9 ADXL345, P1 USB_C_Plug, Q1 NMOS, U1 TMC2209-LA, U2 STM32G431KBU3, U3 AMS1117-3.3, Y1 Crystal_GND24

Commit message: Just chucked whatever is here
Going on holidays and just have an old version but this is backup skibidi 67
Parts:
- added H1: m1.5, Library:MountingHole_M1.5, F.Cu at (214.7, 62.3)
- added H2: m1.5, Library:MountingHole_M1.5, F.Cu at (178.0, 100.0)
- added H3: m1.5, Library:MountingHole_M1.5, F.Cu at (175.0, 62.2)
- added SW1: SW_SPST, Connector_PinHeader_2.54mm:PinHeader_1x02_P2.54mm_Vertical, F.Cu at (199.4, 76.2)
- R100, R9: footprint Resistor_SMD:R_1218_3246Metric -> Resistor_SMD:R_1206_3216Metric
- moved C22 58.4 mm to (192.7, 77.9)
- moved C3 53.6 mm to (211.6, 78.0), turned to 90 degrees
- moved C4 46.3 mm to (211.5, 87.7), turned to -90 degrees
- moved J9 38.4 mm to (215.5, 73.9), turned to 90 degrees
- moved J2 32.9 mm to (185.8, 84.6)
- moved R11 31.6 mm to (188.8, 84.4)
- moved R100 2.11 mm to (209.1, 75.4)
- moved C5 2.11 mm to (207.0, 88.0)
- moved C6 2.11 mm to (205.5, 82.8)
- moved C8 2.11 mm to (208.6, 80.0)
- moved J1 2.11 mm to (215.0, 87.3)
- moved R2 2.11 mm to (204.9, 86.0)
- moved R3 2.11 mm to (208.0, 88.0)
- moved R4 2.11 mm to (209.5, 88.0)
- moved R6 2.11 mm to (211.0, 79.8)
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Routing:
- net Net-(J11-Pin_1): track 11.0 -> 0.95 mm
Other:
- board outline added: 49.6 x 43.6 mm
- board text added: "ABL"
- board text added: "EXF"
- board text added: "FILA"
- board text added: "HOT"
- board text added: "PCF"
- board text added: "m1.5 screws"

Commit message: e
e
Parts:
- removed C14, C15: 10uF, Capacitor_SMD:C_0603_1608Metric
- removed C27: 4.7uF 50V, Capacitor_SMD:C_1206_3216Metric
- removed D2: D, Diode_SMD:D_SOD-123F
- removed Q1: NMOS, Library:PPAK-8L-NumberingFixed
- removed R22: 4.7k, Resistor_SMD:R_0402_1005Metric
- removed R242: 10k, Resistor_SMD:R_0402_1005Metric
- removed U3: AMS1117-3.3, Package_TO_SOT_SMD:SOT-223-3_TabPin2
- added C1: 100nF, PCM_JLCPCB:C_0402, F.Cu at (218.5, 85.4)
- added C11: 4.7uF, PCM_JLCPCB:C_1206, F.Cu at (206.6, 95.5)
- added C9: 1uF, PCM_JLCPCB:C_0402, F.Cu at (193.5, 95.8)
- added D4: DSK26, PCM_JLCPCB:D_SOD-123FL, F.Cu at (202.0, 95.5)
- added J12: THO, Connector_JST:JST_XH_B2B-XH-A_1x02_P2.50mm_Vertical, F.Cu at (214.2, 79.9)
- added J13: HE, Connector_JST:JST_XH_B2B-XH-A_1x02_P2.50mm_Vertical, F.Cu at (207.6, 65.9)
- added PN1: ~, PCM_JLCPCB:Part_Num_JLCPCB, F.Cu at (183.5, 96.1)
- added Q2: AO3400A, PCM_JLCPCB:Q_SOT-23, F.Cu at (201.4, 65.1)
- added R26: 4.7kΩ, PCM_JLCPCB:R_0402, F.Cu at (197.3, 95.8)
- added R27: 10Ω, PCM_JLCPCB:R_0402, F.Cu at (201.3, 69.0)
- added R28: 10kΩ, PCM_JLCPCB:R_0402, F.Cu at (198.9, 93.8)
- added R29: 4.7kΩ, PCM_JLCPCB:R_0402, F.Cu at (195.3, 95.8)
- added R30: 10kΩ, PCM_JLCPCB:R_0402, F.Cu at (202.3, 69.0)
- added R31: 4.7kΩ, PCM_JLCPCB:R_0402, F.Cu at (210.8, 77.8)
- added U4: USBLC6-2SC6, Package_TO_SOT_SMD:SOT-23-6, F.Cu at (193.8, 71.9)
- added U5: TLV75733PDBV, Package_TO_SOT_SMD:SOT-23-5, F.Cu at (189.6, 87.6)
- added U6: 74LVC1G17, PCM_JLCPCB:SOT-23-5_L3.0-W1.7-P0.95-LS2.8-BR, F.Cu at (182.2, 71.7)
- C12: value 100nF -> 4.7uF; footprint Capacitor_SMD:C_0402_1005Metric -> PCM_JLCPCB:C_1206
- C13: value 4.7uF 50V -> 100nF; footprint Capacitor_SMD:C_1206_3216Metric -> PCM_JLCPCB:C_0402
- C16, C23: footprint Capacitor_SMD:C_0402_1005Metric -> PCM_JLCPCB:C_0402
- C17: value 100nF -> 1uF; footprint Capacitor_SMD:C_0402_1005Metric -> PCM_JLCPCB:C_0402
- C18: value 10uF -> 1uF; footprint Capacitor_SMD:C_0603_1608Metric -> PCM_JLCPCB:C_0402
- C19: value 10nF -> 10uF; footprint Capacitor_SMD:C_0402_1005Metric -> PCM_JLCPCB:C_0603
- C20: value 1uF -> 10nF; footprint Capacitor_SMD:C_0201_0603Metric -> PCM_JLCPCB:C_0402
- C21: footprint Capacitor_SMD:C_0201_0603Metric -> PCM_JLCPCB:C_0402
- C22: value 100nF -> 30pF; footprint Capacitor_SMD:C_0402_1005Metric -> PCM_JLCPCB:C_0402
- C24: value 30pF -> 1uF; footprint Capacitor_SMD:C_0402_1005Metric -> PCM_JLCPCB:C_0402
- C3, C4, C5: value 100nF 50V -> 100nF; footprint Capacitor_SMD:C_0402_1005Metric -> PCM_JLCPCB:C_0402
- C6: value 4.7uF -> 22nF; footprint Capacitor_SMD:C_0201_0603Metric -> PCM_JLCPCB:C_0402
- C7: value 100nF 50V -> 4.7uF; footprint Capacitor_SMD:C_0402_1005Metric -> PCM_JLCPCB:C_1206
- C8: value 22nF 50V -> 100nF; footprint Capacitor_SMD:C_0402_1005Metric -> PCM_JLCPCB:C_0402
- D1: value D -> DSK26; footprint Diode_SMD:D_SOD-123F -> PCM_JLCPCB:D_SOD-123FL
- J10: footprint Connector_JST:JST_XH_B5B-XH-A_1x05_P2.50mm_Vertical -> Connector_PinHeader_2.54mm:PinHeader_1x05_P2.54mm_Vertical
- J11: value HT_THO -> EXTR_FIL; footprint Connector_JST:JST_XH_B4B-XH-A_1x04_P2.50mm_Vertical -> Connector_PinHeader_2.54mm:PinHeader_1x02_P2.54mm_Vertical
- J14: value Conn_01x08_Pin -> FPC_FILAMENT_SENSOR; footprint Connector_FFC-FPC:Amphenol_F32Q-1A7x1-11008_1x08-1MP_P0.5mm_Horizontal -> Connector_FFC-FPC:Hirose_FH12-8S-0.5SH_1x08-1MP_P0.50mm_Horizontal
- J9: footprint Connector_JST:JST_XH_B4B-XH-A_1x04_P2.50mm_Vertical -> Connector_PinHeader_2.54mm:PinHeader_1x04_P2.54mm_Vertical
- R11: value 10kR -> 10kΩ; footprint Resistor_SMD:R_0402_1005Metric -> PCM_JLCPCB:R_0402
- R16: value 10R -> 4.7kΩ; footprint Resistor_SMD:R_0402_1005Metric -> PCM_JLCPCB:R_0402
- R17: value 20kR -> 2.2kΩ; footprint Resistor_SMD:R_0402_1005Metric -> Resistor_SMD:R_0603_1608Metric
- R18: value 4.7kR -> 2.2kΩ; footprint Resistor_SMD:R_0402_1005Metric -> Resistor_SMD:R_0603_1608Metric
- R19, R20: value 2.37kR -> 10kΩ; footprint Resistor_SMD:R_0402_1005Metric -> PCM_JLCPCB:R_0402
- R2, R5: value 20ko -> 20kΩ; footprint Resistor_SMD:R_0402_1005Metric -> PCM_JLCPCB:R_0402
- R21: value 10k -> 100Ω; footprint Resistor_SMD:R_0402_1005Metric -> PCM_JLCPCB:R_0402
- R23: value 10k -> 4.7kΩ; footprint Resistor_SMD:R_0402_1005Metric -> PCM_JLCPCB:R_0402
- R24: value 10k -> 10kΩ; footprint Resistor_SMD:R_0402_1005Metric -> PCM_JLCPCB:R_0402
- R25: value 4.7k -> 10kΩ; footprint Resistor_SMD:R_0402_1005Metric -> PCM_JLCPCB:R_0402
- R3, R4, R6: value 100o -> 100Ω; footprint Resistor_SMD:R_0402_1005Metric -> PCM_JLCPCB:R_0402
- R7: value 20ko -> 10kΩ; footprint Resistor_SMD:R_0402_1005Metric -> PCM_JLCPCB:R_0402
- R8: value 100o -> 20kΩ; footprint Resistor_SMD:R_0402_1005Metric -> PCM_JLCPCB:R_0402
- moved C12 42.9 mm to (215.6, 66.2), turned to 180 degrees
- moved C3 40.6 mm to (171.5, 84.6), turned to 180 degrees
- moved R100 36.5 mm to (173.2, 82.1), turned to 180 degrees
- moved R3 35.6 mm to (172.4, 86.6), turned to 0 degrees
- moved J1 35.4 mm to (180.8, 78.1), turned to 180 degrees
- moved C7 35.3 mm to (174.7, 92.0)
- moved J9 35.1 mm to (190.2, 98.2)
- moved D3 34.9 mm to (216.2, 85.9)
- moved C5 34.6 mm to (172.4, 89.4), turned to 180 degrees
- moved C6 34.0 mm to (171.9, 88.0), turned to 90 degrees
- moved R18 33.5 mm to (214.0, 87.6), turned to 180 degrees
- moved R5 32.5 mm to (172.4, 85.7), turned to 180 degrees
- moved U1 31.8 mm to (177.4, 87.4), turned to 0 degrees
- moved R17 30.8 mm to (217.6, 88.4), turned to 90 degrees
- moved J7 30.4 mm to (209.2, 73.0), turned to 0 degrees
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Connections:
- C12 pad 1: /heaters/THERMISTER -> +24V
- C13 pad 1: +24V -> +3V3
- C18 pad 1: +3V3 -> +3V3A
- C19 pad 1: +3V3A -> +3V3
- C22 pad 1: Net-(SW1-B) -> Net-(U2-PF1)
- C24 pad 1: Net-(U2-PF1) -> GND
- C24 pad 2: GND -> VBUS
- C5 pad 1: +3V3 -> Net-(U1-VCP)
- C5 pad 2: GND -> +24V
- C6 pad 1: +5V -> Net-(U1-CPI)
- C6 pad 2: GND -> Net-(U1-CPO)
- C7 pad 1: Net-(U1-VCP) -> +5V
- C7 pad 2: +24V -> GND
- C8 pad 1: Net-(U1-CPI) -> +3V3
- C8 pad 2: Net-(U1-CPO) -> GND
- D1 pad 1: VBUS -> +24V
- J10 pad 1: GND3 -> GND
- J10 pad 3: GND3 -> GND
- J11 pad 1: Net-(J11-Pin_1) -> /reversed_filament_sensor/SNS1
- J11 pad 2: GND -> /reversed_filament_sensor/SNS2
- J14 pad 1: Net-(J14-Pin_1) -> +3V3
- J14 pad 2: Net-(J14-Pin_1) -> +3V3
- J14 pad 3: GND -> /reversed_filament_sensor/SNS1
- J14 pad 4: /mcu/FILA_SENSOR_1ADC -> unconnected-(J14-Pin_4-Pad4)
- J14 pad 5: /mcu/FILA_SENSOR_1ADC -> /reversed_filament_sensor/SNS2
- J14 pad 6: /mcu/FILA_SENSOR_1ADC -> /reversed_filament_sensor/SNS3
- J14 pad 7: +3V3 -> GND
- J14 pad 8: +3V3 -> GND
- P1 pad A6: /communications/USB_D+ -> /communications/USB_PORT_D+
- P1 pad A7: /communications/USB_D- -> /communications/USB_PORT_D-
- P1 pad B6: (no net) -> /communications/USB_PORT_D+
- P1 pad B7: (no net) -> /communications/USB_PORT_D-
- P1 pad S1: GND -> (no net)
- R11 pad 1: Net-(J2-Pin_2) -> +3V3
- R11 pad 2: Net-(U2-PB8) -> Net-(SW1-B)
- R16 pad 1: /heaters/HOTEND_PWM -> +3.3VADC
- R16 pad 2: Net-(Q1-G) -> Net-(J12-Pin_1)
- R17 pad 1: /heaters/HOTEND_PWM -> /heaters/THERMISTER
- R17 pad 2: GND -> Net-(D3-K-Pad3)
- R18 pad 1: +3.3VADC -> Net-(D3-K-Pad3)
- R18 pad 2: Net-(J11-Pin_1) -> Net-(J12-Pin_1)
- R19 pad 1: Net-(J11-Pin_1) -> Net-(J6-Pin_2)
- R19 pad 2: Net-(D3-K-Pad3) -> +3V3
- R20 pad 1: Net-(D3-K-Pad3) -> /fans/EXTR_FAN_TACH
- R20 pad 2: /heaters/THERMISTER -> Net-(J6-Pin_2)
- R21 pad 1: +3V3 -> /mcu/EXTRUDER_DIAG
- R21 pad 2: Net-(J7-Pin_1) -> Net-(U1-DIAG)
- R23 pad 1: /fans/EXTR_FAN_TACH -> /fans/EXTR_FAN_PWM
- R23 pad 2: Net-(J6-Pin_2) -> GND
- R24 pad 1: +3V3 -> Net-(J7-Pin_1)
- R24 pad 2: Net-(J6-Pin_2) -> +3V3
- R25 pad 1: /fans/EXTR_FAN_PWM -> /fans/PART_FAN_TACH
- R25 pad 2: GND -> Net-(J7-Pin_1)
- R3 pad 1: /mcu/EXTRUDER_STEP -> /mcu/EXTRUDER_ENABLE
- R3 pad 2: Net-(U1-STEP) -> Net-(U1-~{EN})
- R4 pad 1: /mcu/EXTRUDER_DIR -> Net-(U1-STEP)
- R4 pad 2: Net-(U1-DIR) -> /mcu/EXTRUDER_STEP
- R5 pad 1: GND -> Net-(U1-~{EN})
- R5 pad 2: Net-(U1-CLK) -> +3V3
- R6 pad 1: /mcu/EXTRUDER_ENABLE -> /mcu/EXTRUDER_DIR
- R6 pad 2: Net-(U1-~{EN}) -> Net-(U1-DIR)
- R7 pad 1: Net-(U1-~{EN}) -> Net-(J2-Pin_2)
- R7 pad 2: +3V3 -> Net-(U2-PB8)
- R8 pad 1: Net-(U1-DIAG) -> GND
- R8 pad 2: /mcu/EXTRUDER_DIAG -> Net-(U1-CLK)
- U2 pad 10: /mcu/EXTRUDER_DIAG -> /fans/EXTR_FAN_TACH
- U2 pad 11: /mcu/EXTRUDER_ENABLE -> /heaters/THERMISTER
- U2 pad 12: /mcu/EXTRUDER_DIR -> /fans/PART_FAN_PWM
- U2 pad 13: /mcu/EXTRUDER_STEP -> /fans/PART_FAN_TACH
- U2 pad 26: /fans/PART_FAN_PWM -> /mcu/FILAMENT_SENSOR
- U2 pad 27: /fans/PART_FAN_TACH -> /mcu/EXTRUDER_STEP
- U2 pad 28: /fans/EXTR_FAN_PWM -> /mcu/EXTRUDER_DIAG
- U2 pad 29: /fans/EXTR_FAN_TACH -> /mcu/EXTRUDER_ENABLE
- U2 pad 5: /mcu/BIQU_BL_SERVO -> /mcu/EXTRUDER_DIR
- U2 pad 6: /mcu/BIQU_BL_PROBE -> unconnected-(U2-PA1-Pad6)
- U2 pad 7: /mcu/FILA_SENSOR_1ADC -> /mcu/BIQU_BL_PROBE
- U2 pad 8: /mcu/FILA_SENSOR_2 -> /mcu/BIQU_BL_SERVO
- U2 pad 9: /heaters/THERMISTER -> /fans/EXTR_FAN_PWM
Routing:
- net GND: track 1.73 -> 47.5 mm
- net VBUS: track 0.00 -> 45.2 mm
- net /mcu/EXTRUDER_ENABLE: track 0.00 -> 40.4 mm
- net /mcu/BIQU_BL_PROBE: track 0.00 -> 30.0 mm
- net /mcu/EXTRUDER_DIAG: track 0.00 -> 28.4 mm
- net /mcu/EXTRUDER_STEP: track 0.00 -> 23.6 mm
- net /mcu/FILAMENT_SENSOR: track 0.00 -> 21.8 mm, vias 0 -> 2
- net /mcu/BIQU_BL_SERVO: track 0.00 -> 21.5 mm
- net /mcu/ADXL_SDA: track 0.00 -> 20.2 mm
- net /fans/EXTR_FAN_PWM: track 0.00 -> 20.1 mm
- net /heaters/THERMISTER: track 0.00 -> 20.1 mm
- net /mcu/ADXL_SCK: track 0.00 -> 19.8 mm, vias 0 -> 2
- net +3V3: track 0.00 -> 16.8 mm
- net /fans/EXTR_FAN_TACH: track 0.00 -> 14.2 mm
- net +24V: track 16.0 -> 29.5 mm, vias 0 -> 4
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- added copper zone on B.Cu, net GND
Other:
- board text added: "ADXL I2C"
- board text added: "EXTR MOTOR"
- board text added: "FILSNS"
- board text added: "HE"
- board text added: "HE FAN"
- board text added: "Keep Cool area (Suggestion)"
- board text added: "PC FAN"
- board text added: "PROB"
- board text added: "Stick over edge acceptable"
- board text added: "THO"
- board text added: "WRONG FOOTPRINT"
- board text removed: "ABL"
- board text removed: "EXF"
- board text removed: "HOT"
- board text removed: "PCF"

Commit message: e
e
Parts:
- U1: footprint Package_DFN_QFN:VQFN-28-1EP_5x5mm_P0.5mm_EP3.7x3.7mm_ThermalVias -> TMC2209-LA:TMC2209-LargerVias
- moved C3 0.12 mm to (171.6, 84.6)
- moved R31 0.06 mm to (210.8, 77.8)
Connections:
- H1 pad 1: Net-(H1-Pad1) -> unconnected-(H1-Pad1)
- H2 pad 1: Net-(H1-Pad1) -> unconnected-(H2-Pad1)
- H3 pad 1: Net-(H1-Pad1) -> unconnected-(H3-Pad1)
Routing:
- net +3V3: track 16.8 -> 163.0 mm, vias 0 -> 9
- net GND: track 47.5 -> 138.6 mm, vias 0 -> 20
- net +24V: track 29.5 -> 87.8 mm, vias 4 -> 7
- net /mcu/EXTRUDER_TX: track 1.64 -> 34.9 mm, vias 0 -> 2
- net /mcu/EXTRUDER_DIR: track 1.24 -> 28.1 mm, vias 1 -> 6
- net VBUS: track 45.2 -> 69.0 mm, vias 0 -> 4
- net /fans/PART_FAN_PWM: track 4.75 -> 17.2 mm
- net /fans/PART_FAN_TACH: track 0.00 -> 9.96 mm
- net Net-(SW1-B): track 2.38 -> 9.38 mm, vias 0 -> 1
- net Net-(J2-Pin_2): track 0.00 -> 5.84 mm
- net /mcu/EXTRUDER_RX: track 0.00 -> 3.47 mm
- net Net-(U2-PB8): track 0.00 -> 2.35 mm
- net /heaters/HOTEND_PWM: track 12.8 -> 13.9 mm, vias 0 -> 2

Commit message: e
e
Parts:
- J10: footprint Connector_PinHeader_2.54mm:PinHeader_1x05_P2.54mm_Vertical -> Connector_JST:JST_XH_B5B-XH-A_1x05_P2.50mm_Vertical
- moved PN1 16.1 mm to (192.4, 109.5)
- moved C9 10.5 mm to (183.5, 92.7), turned to 180 degrees
- moved R26 10.5 mm to (187.3, 92.7)
- moved R29 10.4 mm to (185.4, 92.7), turned to 180 degrees
- moved R28 9.87 mm to (206.2, 87.2), turned to 180 degrees
- moved J9 8.81 mm to (182.0, 95.0)
- moved U4 3.55 mm to (197.1, 73.3), turned to -45 degrees
- moved J11 3.30 mm to (172.9, 70.3)
- moved J10 2.10 mm to (187.5, 99.7), turned to 0 degrees
- moved C12 1.97 mm to (214.2, 67.6), turned to -90 degrees
- moved D1 1.43 mm to (216.6, 67.7), turned to -90 degrees
- moved Q2 1.03 mm to (201.9, 66.0)
- moved C24 0.93 mm to (190.0, 85.0)
- moved C21 0.63 mm to (190.7, 90.3)
- moved U5 0.63 mm to (190.2, 87.6)
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Connections:
- U4 pad 1: /communications/USB_PORT_D+ -> /communications/USB_PORT_D-
- U4 pad 3: /communications/USB_PORT_D- -> /communications/USB_PORT_D+
- U4 pad 4: /communications/USB_D- -> /communications/USB_D+
- U4 pad 6: /communications/USB_D+ -> /communications/USB_D-
Routing:
- net +3V3: track 163.0 -> 49.2 mm, vias 9 -> 8
- net GND: track 138.6 -> 103.5 mm
- net Net-(J1-Pin_1): track 10.6 -> 0.00 mm
- net VBUS: track 69.0 -> 78.0 mm, vias 4 -> 3
- net Net-(J1-Pin_4): track 8.05 -> 0.00 mm
- net /mcu/EXTRUDER_DIR: track 28.1 -> 20.8 mm, vias 6 -> 2
- net /mcu/EXTRUDER_STEP: track 23.6 -> 18.6 mm
- net /mcu/BIQU_BL_SERVO: track 21.5 -> 26.1 mm
- net /communications/USB_D+: track 11.8 -> 8.02 mm, vias 2 -> 0
- net /communications/USB_D-: track 12.1 -> 8.40 mm, vias 2 -> 0
- net /mcu/BIQU_BL_PROBE: track 30.0 -> 33.4 mm
- net /communications/USB_PORT_D+: track 5.47 -> 8.66 mm
- net /mcu/EXTRUDER_DIAG: track 28.4 -> 25.3 mm
- net /fans/EXTR_FAN_TACH: track 14.2 -> 16.9 mm
- net /fans/EXTR_FAN_PWM: track 20.1 -> 22.8 mm
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- added copper zone on In2.Cu, net +3V3
- added copper zone on In1.Cu, net GND
- added copper zone on F.Cu, net Net-(J1-Pin_1)
- added copper zone on F.Cu, net Net-(J1-Pin_2)
- added copper zone on F.Cu, net Net-(J1-Pin_3)
- added copper zone on F.Cu, net Net-(J1-Pin_4)
Other:
- copper layers 2 -> 4
- board text added: "MOTOR"
- board text added: "PROBE"
- board text removed: "EXTR MOTOR"
- board text removed: "PROB"
