File: Hardware Files/A1-Toolhead-Board/communications.kicad_sch (KiCad schematic)
At the start: 4 parts, among them P1 USB_C_Plug, U3 AMS1117-3.3

Commit message: Just chucked whatever is here
Going on holidays and just have an old version but this is backup skibidi 67
Other:
- note added: "add usb+- esd protection"
- note added: "get 5a plug, justin case"
- note added: "look into TI one = pera"
Changed lines of the file:
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@@
+		)
+	)
+	(text "get 5a plug, justin case\n"
+		(exclude_from_sim no)
+		(at 111.506 137.16 0)
+		(effects
+			(font
+				(size 1.27 1.27)
+			)
+		)
+	)
+	(text "look into TI one = pera"
+		(exclude_from_sim no)
+		(at 152.908 45.466 0)
+		(effects
+			(font
+				(size 1.27 1.27)
+			)
 		)
 	)
@@
 			)
 		)
+	)
+	(text "add usb+- esd protection"
+		(exclude_from_sim no)
+		(at 106.934 84.582 0)
+		(effects
+			(font
+				(size 1.27 1.27)
+			)
+		)

Commit message: e
e
Parts:
- added C21, C24: 1uF, PCM_JLCPCB:C_0402, symbol PCM_JLCPCB-Capacitors:0402,1uF
- added PN1: (no value), PCM_JLCPCB:Part_Num_JLCPCB, symbol PCM_JLCPCB-Manufacturing:Part Number, PCM_JLCPCB, 0.8x0.15mm
- added U4: USBLC6-2SC6, Package_TO_SOT_SMD:SOT-23-6, symbol Power_Protection:USBLC6-2SC6
- added U5: TLV75733PDBV, Package_TO_SOT_SMD:SOT-23-5, symbol Regulator_Linear:TLV75733PDBV
- C14, C15, U3: now not fitted; now left out of the parts list
- P1: symbol Connector:USB_C_Plug -> Connector:USB_C_Receptacle
Connections:
- net +3V3: now also C21.1, U5.5 (OUT)
- net GND: now also P1.SH (SHIELD), C21.2, C24.1, U4.2 (GND), U5.2 (GND); no longer P1.S1 (SHIELD)
- net USB_D+: now also U4.6 (I/O1); no longer P1.A6 (D+)
- net USB_D-: now also U4.4 (I/O2); no longer P1.A7 (D-)
- net VBUS: now also C24.2, U4.5 (VBUS), U5.1 (IN), U5.3 (EN)
- new net USB_PORT_D+: P1.A6 (D+), P1.B6 (D+), U4.1 (I/O1)
- new net USB_PORT_D-: P1.A7 (D-), P1.B7 (D-), U4.3 (I/O2)
Other:
- note added: "C485517"

Commit message: e
e
Connections:
- net USB_D+: now also U4.4 (I/O2); no longer U4.6 (I/O1)
- net USB_D-: now also U4.6 (I/O1); no longer U4.4 (I/O2)
- net USB_PORT_D+: now also U4.3 (I/O2); no longer U4.1 (I/O1)
- net USB_PORT_D-: now also U4.1 (I/O1); no longer U4.3 (I/O2)
Changed lines of the file:
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@@
-		)
-	)
-	(hierarchical_label "USB_D+"
-		(shape input)
-		(at 163.83 96.52 270)
-		(effects
-			(font
-				(size 1.27 1.27)
-			)
-			(justify right)
 		)
 	)
@@
 	(hierarchical_label "USB_PORT_D-"
 		(shape input)
-		(at 161.29 86.36 90)
+		(at 163.83 86.36 90)
 		(effects
 			(font
@@
 	(hierarchical_label "USB_PORT_D+"
 		(shape input)
-		(at 163.83 86.36 90)
+		(at 161.29 86.36 90)
 		(effects
 			(font
@@
 		)
 	)
-	(hierarchical_label "USB_D-"
+	(hierarchical_label "USB_D+"
 		(shape input)
 		(at 161.29 96.52 270)
 		(effects
 			(font
+				(size 1.27 1.27)
+			)
+			(justify right)
+		)
+	)
+	(hierarchical_label "USB_D-"
+		(shape input)
+		(at 163.83 96.52 270)
+		(effects
+			(font
